File: pcb/kicad/flix_all_in_one.kicad_sch (KiCad schematic)
At the start: 20 parts, among them J1 UJ20-C-H-G-MSMT-2B-P16-TR, J2 BM03B-GHS-TBT_LF__SN__N_, J3 BM02B-GHS-TBT_LF__SN__N_, J4 BM02B-GHS-TBT_LF__SN__N_, J5 BM02B-GHS-TBT_LF__SN__N_, J6 BM02B-GHS-TBT_LF__SN__N_, J7 Conn_01x02_Pin, Q2 SLMT320V4CP, U3 TP4054ST25P, U4 ME6211C33M5

Commit message: update sch structure
Parts:
- removed C1, C2: C, symbol Device:C
- removed D1, D2, D3: SLESD5LM5.0CS, SODFL1608X70N, symbol SLESD5LM5.0CS:SLESD5LM5.0CS
- removed D4: 1N5819HW-7-F, SOD3716X125N, symbol 1N5819HW-7-F:1N5819HW-7-F
- removed J1: UJ20-C-H-G-MSMT-2B-P16-TR, UJ20-C-H-G-MSMT-2B-P16-TR:SAMESKY_UJ20-C-H-G-MSMT-2B-P16-TR, symbol UJ20-C-H-G-MSMT-2B-P16-TR:UJ20-C-H-G-MSMT-2B-P16-TR
- removed J2: BM03B-GHS-TBT_LF__SN__N_, BM03B-GHS-TBT_LF__SN__N_:CONN_BM03B-GHS-TBT_LF__SN__N_, symbol BM03B-GHS-TBT_LF__SN__N_:BM03B-GHS-TBT_LF__SN__N_
- removed J3, J4, J5, J6: BM02B-GHS-TBT_LF__SN__N_, BM02B-GHS-TBT_LF__SN__N_:JST_BM02B-GHS-TBT_LF__SN__N_, symbol BM02B-GHS-TBT_LF__SN__N_:BM02B-GHS-TBT_LF__SN__N_
- removed J7: Conn_01x02_Pin, symbol Connector:Conn_01x02_Pin
- removed Q2: SLMT320V4CP, SOT95P280X110-3N, symbol SLMT320V4CP:SLMT320V4CP
- removed R1, R2: 5k1, symbol Device:R
- removed R3, R4: 100k, symbol Device:R
- removed U3: TP4054ST25P, C382138:SOT-23-5_L2.9-W1.6-P0.95-LS2.8-BL, symbol TP4054ST25P:TP4054ST25P
- removed U4: ME6211C33M5, Package_TO_SOT_SMD:SOT-23-5, symbol Regulator_Linear:ME6211C33M5
Connections:
- no-connect marks 2 -> 0
Other:
- added sheet flix_ESP32_Bridge (flix_ESP32_Bridge.kicad_sch)
- added sheet flix_IMU_Baro_Motor (flix_IMU_Baro_Motor.kicad_sch)
- added sheet flix_IOs_Power (flix_IOs_Power.kicad_sch)
