File: pcb/kicad/flix_IMU_Baro_Motor.kicad_sch (KiCad schematic)
At the start: 2 parts, among them IC2 BMP384, U2 ICM-40609-D

Commit message: updated lib and sch
Parts:
- added Q3, Q4, Q5, Q6: SLT045N03N2N, flix_fp:SLT045N03N2N_PDFN3333-8, symbol SLT045N03N2N:SLT045N03N2N
Connections:
- new net: Q6.1, Q6.2, Q6.3
- new net: Q4.1, Q4.2, Q4.3
- new net: Q3.1, Q3.2, Q3.3
- new net: Q5.1, Q5.2, Q5.3
