File: pcb/kicad/flix_IOs_Power.kicad_sch (KiCad schematic)
At the start: 20 parts, among them J1 UJ20-C-H-G-MSMT-2B-P16-TR, J2 BM03B-GHS-TBT_LF__SN__N_, J3 BM02B-GHS-TBT_LF__SN__N_, J4 BM02B-GHS-TBT_LF__SN__N_, J5 BM02B-GHS-TBT_LF__SN__N_, J6 BM02B-GHS-TBT_LF__SN__N_, J7 Conn_01x02_Pin, Q2 SLMT320V4CP, U3 TP4054ST25P, U4 ME6211C33M5

Commit message: update sch
Parts:
- removed R1, R2: 5k1, symbol Device:R
- added C3, C4: 10uF, Capacitor_SMD:C_0603_1608Metric, symbol Device:C_Small
- added LED1: 150060RS75000, LEDC1608X70N, symbol 150060RS75000:150060RS75000
- added R1, R2: 5k1, Resistor_SMD:R_0603_1608Metric, symbol Device:R_Small
- added R5: 1k, Resistor_SMD:R_0603_1608Metric, symbol Device:R_Small
- added R6: 2k, Resistor_SMD:R_0603_1608Metric, symbol Device:R_Small
- added R7, R8: 100k, Resistor_SMD:R_0603_1608Metric, symbol Device:R_Small
- C1, C2: footprint (none) -> Capacitor_SMD:C_0603_1608Metric; symbol Device:C -> Device:C_Small
- R3, R4: footprint (none) -> Resistor_SMD:R_0603_1608Metric; symbol Device:R -> Device:R_Small
Connections:
- net GND: now also U3.2 (GND), C3.2, C4.2, R1.2, R2.2, R6.2, R8.1
- net VBUS: now also U3.4 (VCC), C4.1, R5.1
- net V_Batt: now also U3.3 (BAT), C3.1, R7.2
- net at J1.A5 (CC1): now also R1.1
- net at J1.B5 (CC2): now also R2.1
- net at U3.1 (~{CHRG}): now also LED1.1 (K)
- net at U3.5 (PROG): now also R6.1
- new net: LED1.2 (A), R5.2
- new net ADC_Vbatt: R7.1, R8.2
Other:
- moved on the sheet: C1, C2, D4, Q2, R3, R4, U3, U4

Commit message: updated lib and sch
Parts:
- C1, C2: value C -> 1uF
Connections:
- net GND: no longer J3.2, J4.2, J5.2
- net Motor_1_N: now reaches J6.2
- new net Motor_2_N: J3.2
- new net Motor_3_N: J4.2
- new net Motor_4_N: J5.2
Changed lines of the file:
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@@
 	)
 	(junction
-		(at 106.68 139.7)
-		(diameter 0)
-		(color 0 0 0 0)
-	)
-	(junction
 		(at 187.96 67.31)
 		(diameter 0)
@@
 	)
 	(junction
-		(at 59.69 139.7)
-		(diameter 0)
-		(color 0 0 0 0)
-	)
-	(junction
 		(at 62.23 77.47)
 		(diameter 0)
@@
 	)
 	(junction
-		(at 106.68 119.38)
-		(diameter 0)
-		(color 0 0 0 0)
-	)
-	(junction
 		(at 87.63 44.45)
 		(diameter 0)
@@
 	(wire
 		(pts
+			(xy 102.87 114.3) (xy 109.22 114.3)
+		)
+		(stroke
+			(width 0)
+			(type default)
+		)
+	)
+	(wire
+		(pts
 			(xy 106.68 119.38) (xy 106.68 121.92)
 		)
@@
 	(wire
 		(pts
+			(xy 55.88 114.3) (xy 62.23 114.3)
+		)
+		(stroke
+			(width 0)
+			(type default)
+		)
+	)
+	(wire
+		(pts
 			(xy 55.88 111.76) (xy 62.23 111.76)
 		)
@@
 	(wire
 		(pts
-			(xy 102.87 134.62) (xy 106.68 134.62)
-		)
-		(stroke
-			(width 0)
-			(type default)
-		)
-	)
-	(wire
-		(pts
 			(xy 97.79 46.99) (xy 97.79 41.91)
 		)
@@
 	(wire
 		(pts
-			(xy 55.88 134.62) (xy 59.69 134.62)
-		)
-		(stroke
-			(width 0)
-			(type default)
-		)
-	)
-	(wire
-		(pts
 			(xy 173.99 135.89) (xy 187.96 135.89)
 		)
@@
 	(wire
 		(pts
-			(xy 106.68 134.62) (xy 106.68 139.7)
-		)
-		(stroke
-			(width 0)
-			(type default)
-		)
-	)
-	(wire
-		(pts
 			(xy 63.5 64.77) (xy 66.04 64.77)
 		)
@@
 	(wire
 		(pts
-			(xy 55.88 114.3) (xy 59.69 114.3)
-		)
-		(stroke
-			(width 0)
-			(type default)
-		)
-	)
-	(wire
-		(pts
 			(xy 62.23 173.99) (xy 62.23 176.53)
 		)
@@
 	(wire
 		(pts
-			(xy 59.69 134.62) (xy 59.69 142.24)
+			(xy 170.18 54.61) (xy 187.96 54.61)
 		)
 		(stroke
@@
 	(wire
 		(pts
-			(xy 170.18 54.61) (xy 187.96 54.61)
+			(xy 208.28 44.45) (xy 208.28 48.26)
 		)
 		(stroke
@@
 	(wire
 		(pts
-			(xy 208.28 44.45) (xy 208.28 48.26)
+			(xy 102.87 134.62) (xy 109.22 134.62)
 		)
 		(stroke
@@
 	(wire
 		(pts
-			(xy 106.68 114.3) (xy 106.68 119.38)
+			(xy 177.8 111.76) (xy 177.8 114.3)
 		)
 		(stroke
@@
 	(wire
 		(pts
-			(xy 177.8 111.76) (xy 177.8 114.3)
+			(xy 228.6 41.91) (xy 233.68 41.91)
 		)
 		(stroke
@@
 	(wire
 		(pts
-			(xy 228.6 41.91) (xy 233.68 41.91)
+			(xy 55.88 134.62) (xy 62.23 134.62)
 		)
 		(stroke
@@
 	(wire
 		(pts
-			(xy 215.9 143.51) (xy 215.9 149.86)
+			(xy 59.69 139.7) (xy 59.69 142.24)
 		)
 		(stroke
@@
 	(wire
 		(pts
-			(xy 58.42 72.39) (xy 62.23 72.39)
+			(xy 215.9 143.51) (xy 215.9 149.86)
 		)
 		(stroke
@@
 	(wire
 		(pts
-			(xy 102.87 114.3) (xy 106.68 114.3)
+			(xy 58.42 72.39) (xy 62.23 72.39)
 		)
 		(stroke
@@
 		)
 	)
+	(label "Motor_1_N"
+		(at 62.23 114.3 0)
+		(effects
+			(font
+				(size 1.27 1.27)
+			)
+			(justify left bottom)
+		)
+	)
 	(label "V_Bus"
 		(at 118.11 36.83 0)
@@
 		)
 	)
+	(label "Motor_2_N"
+		(at 62.23 134.62 0)
+		(effects
+			(font
+				(size 1.27 1.27)
+			)
+			(justify left bottom)
+		)
+	)
 	(label "5V_In"
 		(at 114.3 170.18 0)
@@
 		)
 	)
+	(label "Motor_4_N"
+		(at 109.22 134.62 0)
+		(effects
+			(font
+				(size 1.27 1.27)
+			)
+			(justify left bottom)
+		)
+	)
 	(label "USB_D_N"
 		(at 118.11 41.91 0)
@@
 		)
 	)
+	(label "Motor_3_N"
+		(at 109.22 114.3 0)
+		(effects
+			(font
+				(size 1.27 1.27)
+			)
+			(justify left bottom)
+		)
+	)
 	(label "Motor_4_P"
 		(at 109.22 132.08 0)
@@
 			)
 		)
-		(property "Value" "C"
+		(property "Value" "1uF"
 			(at 207.01 59.6899 0)
 			(show_name no)
@@
 			)
 		)
-		(property "Value" "C"
+		(property "Value" "1uF"
 			(at 236.22 49.5299 0)
 			(show_name no)
@@
 	)
 	(group ""
+		(members "00b72930-8b39-4022-8a72-68a6aa723ed3" "089cf39a-6919-41f5-9e41-77494f9c5150"
+			"0c7d3743-b8ac-4582-9d02-398ad024a209" "10803a83-efa9-4a18-9165-4f962d986d01"
+			"19055f50-3710-4e00-8212-a3163e474eeb" "19fc35c5-9885-411f-b24e-2e4ea0e61718"
+			"21e76024-23df-44fa-b7e3-f96655c43fd1" "2360997d-5ffd-4608-9443-e21a58933168"
+			"2772998b-8e15-4d35-9521-f7482d43009d" "2abd998b-94ae-4d9e-a909-48128a55a1af"
+			"2b88b3e8-ff38-4881-ad9b-3a663df8b0a4" "2f3c3f0a-478d-4907-a259-d4dd523a91f4"
+			"3f1fbb2e-253a-461f-8750-5da097865ce4" "51426d21-c444-4eca-acff-63e2a8083d4b"
+			"57af7be2-cea7-410a-8240-3c506615de11" "5af5a1d8-93d6-4a3e-9371-de64461cdfa7"
+			"60ef2a57-90b6-428b-8071-d6557ae359ff" "631ab050-b242-4eff-a479-e91579f8ec00"
+			"9c367974-8f47-4d4e-b93a-ca2156cc2f88" "ad590bdf-386e-4e82-bb32-cf818acdef05"
+			"b12c8d38-9d36-4ab1-9534-4f061f8504c8" "b7c3b851-ab3c-4e4e-8675-03a417eb3967"
+			"b9111a3b-082e-4b1c-8904-896fb5ddf6eb" "d08189fa-9455-4c06-8c49-73bb429f8403"
+			"da255686-c97b-475c-a257-8ad534c4def6" "dc91c53f-d137-4bdd-ba1a-1ad4a9b4295f"
+			"dee6f8a2-cff7-4a70-abb4-8dbb545890c5" "e2d06093-654c-4cd1-8766-44909178b1c1"
+			"e3b6db22-5f08-4cba-ae3a-92c6ab63599a" "e58f715c-3db6-4bff-8212-c3bb586c385f"
+			"eacfcf42-9711-44a1-88dc-8fe7b0a9c2a7" "ed033d0d-4f90-4790-b1ca-a93dca8639b0"
+			"ffcaa704-33d8-495f-9b24-49541b4e4d55"
+		)
+	)
+	(group ""
 		(members "05d78e7b-813d-43e9-a150-e59eb9596aa0" "0901a591-629c-4f83-8c2c-a24ce8c0f9f4"
 			"09451e24-7595-4e4b-9e7d-ac72475767a1" "13aef2fc-cf6d-4faa-8d6b-a96533ed4a4c"
@@
 		)
 	)
-	(group ""
-		(members "00b72930-8b39-4022-8a72-68a6aa723ed3" "089cf39a-6919-41f5-9e41-77494f9c5150"
-			"0c7d3743-b8ac-4582-9d02-398ad024a209" "10803a83-efa9-4a18-9165-4f962d986d01"
-			"14ab9815-87bc-4ae6-bc43-7c668e676246" "19fc35c5-9885-411f-b24e-2e4ea0e61718"
-			"21e76024-23df-44fa-b7e3-f96655c43fd1" "2360997d-5ffd-4608-9443-e21a58933168"
-			"2772998b-8e15-4d35-9521-f7482d43009d" "2982c1e4-3a03-4ec1-801c-d125050f59df"
-			"2b88b3e8-ff38-4881-ad9b-3a663df8b0a4" "2f3c3f0a-478d-4907-a259-d4dd523a91f4"
-			"3b034034-b36c-46eb-aea6-4f48129bb80c" "3f1fbb2e-253a-461f-8750-5da097865ce4"
-			"4b620441-ffb9-40e4-b382-f5472036cbf4" "4bbeff22-4559-44a5-aee8-dbcb391bbbef"
-			"5af5a1d8-93d6-4a3e-9371-de64461cdfa7" "5c9cddd3-8933-49f8-b472-29b1d89b1c45"
-			"60ef2a57-90b6-428b-8071-d6557ae359ff" "94ef4c53-a0f1-4eb8-8db5-8a70e04898b2"
-			"9c367974-8f47-4d4e-b93a-ca2156cc2f88" "ad590bdf-386e-4e82-bb32-cf818acdef05"
-			"b7c3b851-ab3c-4e4e-8675-03a417eb3967" "c4388dcd-e767-4885-9d90-be203abd5f6c"
-			"d08189fa-9455-4c06-8c49-73bb429f8403" "de5f880d-1ff1-4fbc-a4f3-ff7619d21d75"
-			"dee6f8a2-cff7-4a70-abb4-8dbb545890c5" "e2d06093-654c-4cd1-8766-44909178b1c1"
-			"e3b6db22-5f08-4cba-ae3a-92c6ab63599a" "e58f715c-3db6-4bff-8212-c3bb586c385f"
-			"eacfcf42-9711-44a1-88dc-8fe7b0a9c2a7" "ed033d0d-4f90-4790-b1ca-a93dca8639b0"
-			"ffcaa704-33d8-495f-9b24-49541b4e4d55"
-		)
-	)
